File: MACH HARDWARE/VeloR V2.kicad_sch (KiCad schematic)
At the start: 74 parts, among them J1 Conn_01x07_Pin, J2 INICIO, J4 Conn_01x02_Pin, J5 OLED, J6 USB_B_Mini, J7 Conn_01x04_Pin, M1-A1 Conn_01x02_Pin, M100 Motor_DC, M2-A1 Conn_01x02_Pin, M2-A2 Conn_01x02_Pin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

Commit message: Add files via upload
Parts:
- removed J1: Conn_01x07_Pin, Connector_JST:JST_XH_S7B-XH-A_1x07_P2.50mm_Horizontal, symbol Connector:Conn_01x07_Pin
- added J3: Conn_01x10_Pin, Connector_JST:JST_XH_S10B-XH-A_1x10_P2.50mm_Horizontal, symbol Connector:Conn_01x10_Pin
Connections:
- net SCL is gone; now on net SS: J5.2 (Pin_2), U4.28 ((PCINT13/SCL/ADC5)PC5)
- net 3V3: now also J3.1 (Pin_1)
- net CHA: now also U4.19 (ADC6), J3.2 (Pin_2); no longer U4.22 (ADC7)
- net CHB: now also U4.22 (ADC7), J3.3 (Pin_3); no longer U4.23 ((PCINT8/ADC0)PC0)
- net CHC: now also U4.23 ((PCINT8/ADC0)PC0), J3.4 (Pin_4); no longer U4.24 ((PCINT9/ADC1)PC1)
- net CHD: now also U4.24 ((PCINT9/ADC1)PC1), J3.5 (Pin_5); no longer U4.25 ((PCINT10/ADC2)PC2)
- net GND: now also J3.10 (Pin_10)
- net LED_1: now also U4.11 ((PCINT23/AIN1)PD7); no longer U4.32 ((PCINT18/INT0)PD2)
- net SS: now also J3.9 (Pin_9); no longer U4.26 ((PCINT11/ADC3)PC3)
- net ST: now also U4.32 ((PCINT18/INT0)PD2); no longer U4.19 (ADC6)
- net SDA renamed CHG
- net CHG: now also J3.8 (Pin_8)
- new net CHE: J3.6 (Pin_6), U4.25 ((PCINT10/ADC2)PC2)
- new net CHF: J3.7 (Pin_7), U4.26 ((PCINT11/ADC3)PC3)
Other:
- note added: "ARRAY 16/8 SENSORS"
- note added: "PBO=D8 PB1=D9=PWM PB2=D10=PWM PB3=D11=PWM PB4=D12 PB5=D13 PB6=XTAL PB7=XTAL"
- note added: "PCO=A0 PC1=A1 PC2=A2 PC3=A3 PC4=A4 PC5=A5 PC6=RST ADC6=A6 ADC7=A7"
- note added: "PDO=D0=TXD PD1=D1=RXD PD2=D2 PD3=D3=PWM PD4=D4 PD5=D5=PWM PD6=D6=PWM PD7=D7"
- note added: "TURBINE"
- note removed: "ARRAY 16 SENSORS"
- note removed: "PBO=D8 PB1=D9=PWM PB2=D10=PWM PB3=D11=PWM PB4=D12 PB5=D13 PB6=XTAL PB7=XTAL ---------- PDO=D0=TXD PD1=D1=RXD PD2=D2 PD3=D3=PWM PD4=D4 PD5=D5=PWM PD6=D6=PWM PD7=D7 ---------- PCO=A0 PC1=A1 PC2=A2 PC3=A3 PC4=A4 PC5=A5 PC6=RESET ADC6=A6 ADC7=A7"
- note removed: "PBO=D8 |PDO=D0=TXD |PC0=A0 PB1=D9=PWM |PD1=D2=RXD |PC1=A1 PB2=D10=PWM |PD2=D2 |PC2=A2 PB3=D11=PWM |PD3=D3=PWM |PC3=A3 PB4=D12 |PD4=D4 |PC4=A4 PB5=D13 |PD5=D5=PWM |PC5=A5 PB6=XTAL |PD6=D6=PWM |PC6=RESET PB7=XTAL |PD7=D7 |ADC6=A6 ADC7=A7"
- moved on the sheet: C20, C21, C4, C6, C7, D4, J4, M2-A2, MINI360, Q1, R1, R10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

Commit message: Add files via upload
Parts:
- removed C11, C14, C17, C18: 100nF, Capacitor_SMD:C_0805_2012Metric_Pad1.18x1.45mm_HandSolder, symbol Device:C_Small
- removed C16, C19: 100nf, Capacitor_SMD:C_0805_2012Metric_Pad1.18x1.45mm_HandSolder, symbol Device:C
- removed C20, C21: 100nF, Capacitor_SMD:C_0805_2012Metric_Pad1.18x1.45mm_HandSolder, symbol Device:C
- removed C7: 10uF, Capacitor_SMD:C_1206_3216Metric_Pad1.33x1.80mm_HandSolder, symbol Device:C
- removed D3: 1N5819, RAMLIB:Sod123 DIODE, symbol Diode:1N5819
- removed D4: 1N5819, RamLib:Sod123 DIODE, symbol PCM_Diode_Schottky_AKL:1N5819M
- removed J5: OLED, Connector_PinSocket_2.54mm:PinSocket_1x04_P2.54mm_Vertical, symbol Connector:Conn_01x04_Pin
- removed J6: USB_B_Mini, Connector_USB:USB_Mini-B_Lumberg_2486_01_Horizontal, symbol Connector:USB_B_Mini
- removed MINI360: ~, RAMLIB:Mini360_step-down, symbol Trejo huellas nuevas:MINI_360
- removed U2: CH340C, Package_SO:SOIC-16_3.9x9.9mm_P1.27mm, symbol Interface_USB:CH340C
- removed U7: AMS1117-3.3, Package_TO_SOT_SMD:SOT-223-3_TabPin2, symbol Regulator_Linear:AMS1117-3.3
- removed Y1: Crystal_GND2, Crystal:Resonator_SMD_Murata_CSTxExxV-3Pin_3.0x1.1mm, symbol Device:Crystal_GND2
- added C5, C9: 22pF, Capacitor_SMD:C_0805_2012Metric_Pad1.18x1.45mm_HandSolder, symbol Device:C
- added Y2: Crystal, Crystal:Crystal_HC49-4H_Vertical, symbol Device:Crystal
- J7: footprint Connector_PinHeader_2.54mm:PinHeader_1x04_P2.54mm_Vertical -> Connector_PinHeader_2.54mm:PinHeader_1x04_P2.54mm_Horizontal
Connections:
- net +6V is gone; now on net VCC1: C4.1, U3.3 (VI)
- net 3V3 is gone; now on net +5V: J3.1 (Pin_1)
- net GND: now also C5.2, C9.2
- net IN1: now also U4.14 ((PCINT2/OC1B/~{SS})PB2), U6.2 (IN); no longer U4.13 ((PCINT1/OC1A)PB1), U5.2 (IN)
- net IN2: now also U4.13 ((PCINT1/OC1A)PB1), U5.2 (IN); no longer U4.14 ((PCINT2/OC1B/~{SS})PB2), U6.2 (IN)
- net LED_1: now also U4.2 ((PCINT20/XCK/T0)PD4); no longer U4.11 ((PCINT23/AIN1)PD7)
- net LED_2: now also U4.11 ((PCINT23/AIN1)PD7); no longer U4.2 ((PCINT20/XCK/T0)PD4)
- net Q: now also R5.1; no longer R5.2
- net TUR: now also R5.2; no longer R5.1
- net XTAL1: now also C5.1, Y2.1
- net XTAL2: now also C9.1, Y2.2
- no-connect marks 5 -> 4
Other:
- note removed: "TURBINE"
- moved on the sheet: M2-A2, R1, R28, R5

Commit message: Add files via upload
MACH, TRUBINE, DRIVERS TA6586, CNC MACHINE
Parts:
- removed C1, C10, C12, C13, C2, C8: 100n, Capacitor_SMD:C_0805_2012Metric_Pad1.18x1.45mm_HandSolder, symbol Device:C_Small
- removed R15: 10K, Resistor_SMD:R_1206_3216Metric_Pad1.30x1.75mm_HandSolder, symbol Device:R_Small
- removed R17, R18, R9: 10k, Resistor_SMD:R_1206_3216Metric_Pad1.30x1.75mm_HandSolder, symbol Device:R_Small
- removed R19, R20, R52, R83: 1K, Resistor_SMD:R_1206_3216Metric_Pad1.30x1.75mm_HandSolder, symbol Device:R_Small
- removed U10, U5, U6, U9: BTS7960B, Package_TO_SOT_SMD:TO-263-7_TabPin8, symbol BTS7960B:BTS7960B
- added C1, C160, C166, C2: 100nf, Capacitor_SMD:C_0805_2012Metric_Pad1.18x1.45mm_HandSolder, symbol Device:C
- added C11, C7: 100UF, Capacitor_Tantalum_SMD:CP_EIA-7343-20_Kemet-V, symbol Device:C
- added C14, C44: 100nF, Capacitor_SMD:C_0805_2012Metric_Pad1.18x1.45mm_HandSolder, symbol Device:C
- added D3: 1N4007, Diode_SMD:D_SMA, symbol Diode:1N4007
- added TA6586-1, TA6586-2: (no value), Package_DIP:DIP-8_W7.62mm, symbol New_Library_Triatlón:TA6586
- J4: footprint Connector_AMASS:AMASS_XT30U-F_1x02_P5.0mm_Vertical -> Connector_JST:JST_XH_B3B-XH-A_1x03_P2.50mm_Vertical
- M1-A1, M2-A1, M2-A2: footprint Connector_JST:JST_ZH_B2B-ZR_1x02_P1.50mm_Vertical -> Connector_Hirose:Hirose_DF13-02P-1.25DSA_1x02_P1.25mm_Vertical
Connections:
- net +5V: now also C1.1, C2.1
- net GND: now also C1.2, C11.1, C14.1, C2.2, C44.1, C7.1, TA6586-1.3 (GND), TA6586-2.3 (GND)
- net IN1: now also TA6586-2.1 (E1)
- net IN2: now also TA6586-2.2 (E2)
- net IN3: now also TA6586-1.1 (E1)
- net IN4: now also TA6586-1.2 (E2)
- net VCC: now also C11.2, C14.2, C44.2, C7.2, TA6586-1.4 (VCC), TA6586-2.4 (VCC)
- net VCC1: now also D3.1 (K)
- net M_1A renamed M2
- net M2: now also C166.2, TA6586-2.5 (S2), TA6586-2.6 (S2)
- net M_1B renamed M1
- net M1: now also C166.1, TA6586-2.7 (S1), TA6586-2.8 (S1)
- net M_2A renamed M4
- net M4: now also C160.2, TA6586-1.5 (S2), TA6586-1.6 (S2)
- net M_2B renamed M3
- net M3: now also C160.1, TA6586-1.7 (S1), TA6586-1.8 (S1)
- net Q: no longer names the net of Q1.1 (G), R10.1, R5.1
- net VM-: no longer names the net of M2-A2.1 (Pin_1), Q1.3 (D)
- net VM-: now also D3.2 (A)
Other:
- note removed: "BUTTONS"
- note removed: "MOTOR 1"
- note removed: "MOTOR 2"
- moved on the sheet: C4, C6, H1, J4, M2-A2, R10, R5, SW1A, SW2A, SW3A, SW5A, U3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
