File: MACH HARDWARE/VeloR V2.kicad_pcb (KiCad board)
At the start: 2 copper layers, 100 x 96.5 mm, 73 parts, among them J1 Conn_01x07_Pin, J2 INICIO, J4 Conn_01x02_Pin, J5 OLED, J6 USB_B_Mini, J7 Conn_01x04_Pin, M1-A1 Conn_01x02_Pin, M100 Motor_DC, M2-A1 Conn_01x02_Pin, M2-A2 Conn_01x02_Pin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

Commit message: Add files via upload
Parts:
- removed J1: Conn_01x07_Pin, Connector_JST:JST_XH_S7B-XH-A_1x07_P2.50mm_Horizontal
- added J3: Conn_01x10_Pin, Connector_JST:JST_XH_S10B-XH-A_1x10_P2.50mm_Horizontal, F.Cu at (271.5, 156.4)
- moved C14 17.0 mm to (286.8, 170.2), turned to 0 degrees
- moved C16 5.76 mm to (274.5, 168.0), turned to -90 degrees
- moved U7 3.57 mm to (280.1, 165.4), turned to 180 degrees
- moved C7 3.15 mm to (285.8, 165.4), turned to -90 degrees
- moved C19 2.29 mm to (274.5, 162.8), turned to 90 degrees
- moved C1 0.75 mm to (274.5, 231.8)
- moved C10 0.75 mm to (217.5, 243.8)
- moved C11 0.75 mm to (221.2, 174.8)
- moved C12 0.75 mm to (282.9, 230.7)
- moved C13 0.75 mm to (237.5, 230.7)
- moved C15 0.75 mm to (249.5, 180.0)
- moved C17 0.75 mm to (226.2, 165.5)
- moved C18 0.75 mm to (213.0, 179.2)
- moved C2 0.75 mm to (303.2, 243.0)
- moved C20 0.75 mm to (268.5, 185.4)
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Connections:
- net /SDA renamed /CHG
- J5 pad 2: /SCL -> /SS
- U4 pad 11: unconnected-(U4-(PCINT23/AIN1)PD7-Pad11) -> /LED_1
- U4 pad 19: /ST -> /CHA
- U4 pad 22: /CHA -> /CHB
- U4 pad 23: /CHB -> /CHC
- U4 pad 24: /CHC -> /CHD
- U4 pad 25: /CHD -> /CHE
- U4 pad 26: /SS -> /CHF
- U4 pad 28: /SCL -> /SS
- U4 pad 32: /LED_1 -> /ST
Routing:
- net /SCL: track 48.5 -> 0.00 mm, vias 1 -> 0
- net /SS: track 18.1 -> 62.0 mm, vias 0 -> 1
- net Net-(U4-AREF): track 5.50 -> 22.7 mm
- net /CHF: track 0.00 -> 13.6 mm
- net /CHE: track 0.00 -> 11.9 mm
- net /LED_1: track 12.1 -> 23.2 mm, vias 0 -> 2
- net /CHG: track 52.4 -> 63.0 mm
- net /ST: track 36.0 -> 41.6 mm, vias 0 -> 1
- net 3V3: track 58.8 -> 64.1 mm
- net /TUR: track 21.8 -> 25.7 mm
- net /CHD: track 16.3 -> 12.8 mm
- net +5V: track 143.0 -> 145.9 mm, vias 58 -> 47
- net /CHA: track 17.1 -> 19.9 mm, vias 0 -> 2
- net /CHC: track 17.0 -> 14.5 mm, vias 1 -> 0
- net +6V: track 2.47 -> 0.00 mm, vias 20 -> 15
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
Commit message: Add files via upload
Parts:
- removed C11, C14, C17, C18, C20, C21: 100nF, Capacitor_SMD:C_0805_2012Metric_Pad1.18x1.45mm_HandSolder
- removed C16, C19: 100nf, Capacitor_SMD:C_0805_2012Metric_Pad1.18x1.45mm_HandSolder
- removed C7: 10uF, Capacitor_SMD:C_1206_3216Metric_Pad1.33x1.80mm_HandSolder
- removed D3: 1N5819, RAMLIB:Sod123 DIODE
- removed J5: OLED, Connector_PinSocket_2.54mm:PinSocket_1x04_P2.54mm_Vertical
- removed J6: USB_B_Mini, Connector_USB:USB_Mini-B_Lumberg_2486_01_Horizontal
- removed MINI360: ~, RAMLIB:Mini360_step-down
- removed U2: CH340C, Package_SO:SOIC-16_3.9x9.9mm_P1.27mm
- removed U7: AMS1117-3.3, Package_TO_SOT_SMD:SOT-223-3_TabPin2
- removed Y1: Crystal_GND2, Crystal:Resonator_SMD_Murata_CSTxExxV-3Pin_3.0x1.1mm
- added C5: 22pF, Capacitor_SMD:C_0805_2012Metric_Pad1.18x1.45mm_HandSolder, F.Cu at (252.5, 185.2)
- added C9: 22pF, Capacitor_SMD:C_0805_2012Metric_Pad1.18x1.45mm_HandSolder, F.Cu at (257.5, 185.2)
- added Y2: Crystal, Crystal:Crystal_HC49-4H_Vertical, F.Cu at (252.6, 181.2)
- J7: footprint Connector_PinHeader_2.54mm:PinHeader_1x04_P2.54mm_Vertical -> Connector_PinHeader_2.54mm:PinHeader_1x04_P2.54mm_Horizontal
- moved J2 71.9 mm to (225.8, 174.8), turned to 90 degrees
- moved SW6 45.8 mm to (287.8, 188.5), turned to 180 degrees
- moved C4 45.0 mm to (289.2, 163.3), turned to 0 degrees
- moved C3 40.3 mm to (278.8, 170.2), turned to 0 degrees
- moved U3 40.2 mm to (280.9, 165.6), turned to 180 degrees
- moved M2-A2 39.5 mm to (237.2, 173.1), turned to 0 degrees
- moved C15 34.9 mm to (278.8, 161.0), turned to 0 degrees
- moved C2 32.2 mm to (285.8, 216.0), turned to 0 degrees
- moved L4 27.5 mm to (214.7, 185.1)
- moved R16 27.5 mm to (219.5, 185.1)
- moved L2 27.3 mm to (214.7, 181.8)
- moved R14 27.3 mm to (219.5, 181.8)
- moved C10 27.1 mm to (233.0, 221.5), turned to 180 degrees
- moved L1 27.1 mm to (214.7, 178.5)
- moved R13 27.1 mm to (219.5, 178.5)
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Connections:
- C4 pad 1: +6V -> VCC1
- J3 pad 1: 3V3 -> +5V
- R5 pad 1: /TUR -> /Q
- R5 pad 2: /Q -> /TUR
- U3 pad 3: +6V -> VCC1
- U4 pad 11: /LED_1 -> /LED_2
- U4 pad 13: /IN1 -> /IN2
- U4 pad 14: /IN2 -> /IN1
- U4 pad 2: /LED_2 -> /LED_1
- U4 pad 20: Net-(U4-AREF) -> unconnected-(U4-AREF-Pad20)
- U5 pad 2: /IN1 -> /IN2
- U6 pad 2: /IN2 -> /IN1
Routing:
- net 3V3: track 64.1 -> 0.00 mm, vias 1 -> 0
- net /CHG: track 63.0 -> 12.3 mm, vias 1 -> 0
- net /SS: track 62.0 -> 13.6 mm, vias 1 -> 0
- net /LED_2: track 11.0 -> 53.8 mm, vias 0 -> 2
- net /IN3: track 127.4 -> 86.7 mm, vias 2 -> 0
- net /IN1: track 106.0 -> 68.0 mm
- net GND: track 0.00 -> 38.0 mm, vias 19 -> 15
- net /IN2: track 102.9 -> 67.2 mm, vias 2 -> 0
- net /LED_3: track 23.6 -> 59.0 mm
- net +5V: track 145.9 -> 180.4 mm, vias 47 -> 10
- net VCC: track 1.42 -> 33.9 mm, vias 38 -> 14
- net Net-(U4-AREF): track 22.7 -> 0.00 mm
- net /TUR: track 25.7 -> 5.96 mm, vias 2 -> 0
- net Net-(U10-IS): track 23.1 -> 7.01 mm, vias 2 -> 0
- net Net-(U5-SR): track 22.2 -> 6.68 mm, vias 2 -> 0
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- removed copper zone on B.Cu, net +6V
- removed copper zone on F.Cu, net +6V
- removed copper zone on F.Cu, net /CVBUS
- removed copper zone on F.Cu, net /Q
- removed copper zone on F.Cu, net /RESET
- removed copper zone on F.Cu, net 3V3
Other:
- board text added: "QTR8A DIMENSIONS 67MM X 17MM"
- board text removed: "RXD TXD 0V"
- board text removed: "RXD TXD GND 5V"

Commit message: Add files via upload
MACH, TRUBINE, DRIVERS TA6586, CNC MACHINE
Parts:
- removed C10, C12, C13, C8: 100n, Capacitor_SMD:C_0805_2012Metric_Pad1.18x1.45mm_HandSolder
- removed R15: 10K, Resistor_SMD:R_1206_3216Metric_Pad1.30x1.75mm_HandSolder
- removed R17, R18, R9: 10k, Resistor_SMD:R_1206_3216Metric_Pad1.30x1.75mm_HandSolder
- removed R19, R20, R52, R83: 1K, Resistor_SMD:R_1206_3216Metric_Pad1.30x1.75mm_HandSolder
- removed U10, U5, U6, U9: BTS7960B, Package_TO_SOT_SMD:TO-263-7_TabPin8
- added C11: 100UF, Capacitor_Tantalum_SMD:CP_EIA-7343-20_Kemet-V, F.Cu at (253.0, 228.8)
- added C14: 100nF, Capacitor_SMD:C_0805_2012Metric_Pad1.18x1.45mm_HandSolder, F.Cu at (249.0, 226.8)
- added C160: 100nf, Capacitor_SMD:C_0805_2012Metric_Pad1.18x1.45mm_HandSolder, F.Cu at (232.5, 220.0)
- added C166: 100nf, Capacitor_SMD:C_0805_2012Metric_Pad1.18x1.45mm_HandSolder, F.Cu at (287.8, 220.0)
- added C44: 100nF, Capacitor_SMD:C_0805_2012Metric_Pad1.18x1.45mm_HandSolder, F.Cu at (271.0, 226.8)
- added C7: 100UF, Capacitor_Tantalum_SMD:CP_EIA-7343-20_Kemet-V, F.Cu at (267.0, 228.8)
- added D3: 1N4007, Diode_SMD:D_SMA, F.Cu at (240.0, 173.2)
- added TA6586-1: ~, Package_DIP:DIP-8_W7.62mm, F.Cu at (245.0, 221.9)
- added TA6586-2: ~, Package_DIP:DIP-8_W7.62mm, F.Cu at (282.6, 221.9)
- C1, C2: value 100n -> 100nf
- J4: footprint Connector_AMASS:AMASS_XT30U-F_1x02_P5.0mm_Vertical -> Connector_JST:JST_XH_B3B-XH-A_1x03_P2.50mm_Vertical
- M1-A1, M2-A1, M2-A2: footprint Connector_JST:JST_ZH_B2B-ZR_1x02_P1.50mm_Vertical -> Connector_Hirose:Hirose_DF13-02P-1.25DSA_1x02_P1.25mm_Vertical
- moved C2 54.7 mm to (245.0, 179.5), turned to 90 degrees
- moved C1 47.3 mm to (268.2, 169.0), turned to -45 degrees
- moved D1 46.8 mm to (264.3, 221.5)
- moved D11 46.3 mm to (255.5, 221.5)
- moved R1 43.3 mm to (269.4, 221.5), turned to 180 degrees
- moved R28 43.0 mm to (250.6, 221.5), turned to 0 degrees
- moved C9 15.3 mm to (242.2, 186.0)
- moved M1-A1 13.7 mm to (287.1, 225.3), turned to 0 degrees
- moved M2-A1 11.6 mm to (231.9, 225.2), turned to 0 degrees
- moved L1 10.7 mm to (220.0, 187.8)
- moved L2 10.7 mm to (220.0, 191.0)
- moved L4 10.7 mm to (220.0, 194.3)
- moved R13 10.7 mm to (224.8, 187.8)
- moved R14 10.7 mm to (224.8, 191.0)
- moved R16 10.7 mm to (224.8, 194.3)
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Connections:
- net /Q renamed Net-(Q1-G)
- net /VM- renamed Net-(D3-A)
- C1 pad 1: VCC -> +5V
- C2 pad 1: VCC -> +5V
- M1-A1 pad 1: /M_1B -> /M1
- M1-A1 pad 2: /M_1A -> /M2
- M2-A1 pad 1: /M_2B -> /M3
- M2-A1 pad 2: /M_2A -> /M4
Routing:
- net +5V: track 180.4 -> 134.6 mm, vias 10 -> 4
- net VCC: track 33.9 -> 8.43 mm, vias 14 -> 6
- net /ST: track 30.0 -> 46.0 mm
- net VCC1: track 0.00 -> 12.8 mm, vias 3 -> 4
- net /XTAL2: track 10.7 -> 23.5 mm, vias 0 -> 2
- net Net-(U9-SR): track 11.8 -> 0.00 mm
- net Net-(U6-IS): track 11.1 -> 0.00 mm
- net Net-(U5-IS): track 10.1 -> 0.00 mm
- net Net-(U10-SR): track 9.38 -> 0.00 mm
- net /M_2B: track 9.15 -> 0.00 mm, vias 1 -> 0
- net /M_2A: track 9.15 -> 0.00 mm, vias 1 -> 0
- net /M_1B: track 9.15 -> 0.00 mm, vias 1 -> 0
- net /M_1A: track 9.15 -> 0.00 mm, vias 1 -> 0
- net Net-(U9-IS): track 8.35 -> 0.00 mm
- net /SW3: track 45.9 -> 37.9 mm
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- added copper zone on B.Cu, net /M1
- added copper zone on F.Cu, net /M1
- added copper zone on B.Cu, net /M2
- added copper zone on F.Cu, net /M2
- added copper zone on B.Cu, net /M3
- added copper zone on F.Cu, net /M3
- added copper zone on B.Cu, net /M4
- added copper zone on F.Cu, net /M4
- added copper zone on B.Cu, net Net-(D3-A)
- removed copper zone on B.Cu, net +5V
- removed copper zone on F.Cu, net /M_1A
- removed copper zone on F.Cu, net /M_1B
- removed copper zone on F.Cu, net /M_2A
- removed copper zone on F.Cu, net /M_2B
Other:
- board size 100 x 96.5 mm -> 88 x 94.5 mm

Commit message: Add files via upload
Routing:
- net /LED_2: track 50.5 -> 49.4 mm
